Commit message: hw 3 files

File: urdf/simple_world.urdf (robot description, URDF)
Before this commit: robot test, 8 links, 7 joints
Links:
- added link obs_7, mass 1000.0; collision box size=0.4 0.4 0.2; visual box size=0.4 0.4 0.2
- added link obs_8, mass 1000.0; collision box size=0.05 0.05 0.15; visual box size=0.05 0.05 0.15
- added link obs_9, mass 1000.0; collision box size=0.05 0.05 0.15; visual box size=0.05 0.05 0.15
- added link obs_top, mass 1000.0; collision box size=0.05 0.25 0.05; visual box size=0.05 0.25 0.05
- link obs_1: geometry collision box size=2 2 1; visual box size=2 2 1
- link obs_2: geometry collision box size=0.75 0.75 0.75; visual box size=0.75 0.75 0.75
- link obs_3: geometry collision box size=0.75 0.75 0.75; visual box size=0.75 0.75 0.75
- link obs_4: geometry collision box size=0.5 0.5 0.5; visual box size=0.5 0.5 0.5
Joints:
- added joint join10: type fixed, parent wall_1, child obs_7, origin xyz=0.6 0 0.1 rpy=0 0 0
- added joint join11: type fixed, parent wall_1, child obs_8, origin xyz=0.5 0.1 0.275 rpy=0 0 0
- added joint join12: type fixed, parent wall_1, child obs_9, origin xyz=0.5 -0.1 0.275 rpy=0 0 0
- added joint join13: type fixed, parent wall_1, child obs_top, origin xyz=0.5 0 0.375 rpy=0 0 0
- joint join2: origin xyz=2.5 6.25 0.25 rpy=0 0 0 -> xyz=-3.75 3.75 0 rpy=0 0 0; parent wall_1 -> wall_2
- joint join3: origin xyz=-1.25 2.5 0.25 rpy=0 0 0 -> xyz=-3.75 -3.75 0 rpy=0 0 0; parent wall_1 -> wall_3
- joint join6: origin xyz=3 5 0.25 rpy=0 0 0 -> xyz=3 5 0.375 rpy=0 0 0
- joint join7: origin xyz=0 3 0.125 rpy=0 0 0 -> xyz=0 3 0.25 rpy=0 0 0
